File: firmware/hardware/urzadzenie_badawcze_V2/urzadzenie_badawcze_V2.kicad_sch (KiCad schematic)
At the start: 17 parts, among them IC1 MCP6002-I_P, IC2 LM358P, J1 Conn_01x02, J2 Conn_01x04, J3 Conn_01x02, J8 Conn_01x02, Q1 IRLZ44N, Q2 BC547

Commit message: chore: sync repository with current workspace layout
Parts:
- R1: value R 200K -> R 100K
Changed lines of the file:
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@@
 			)
 		)
-		(property "Value" "R 200K"
+		(property "Value" "R 100K"
 			(at 225.552 110.236 90)
 			(effects
