File: hardware/PCB/PCB V2.1/piezotesterV2.1/piezotesterV2.1.kicad_pcb (KiCad board)
At the start: 2 copper layers, 119.3 x 97.3 mm, 49 parts, among them IC1 MCP6002-I_P, IC2 LM358P, IC3 LM2596S-5.0_NOPB, IC4 LP2950-33LPRE3, J1 Conn_01x02, J2 Conn_01x04, J8 Conn_01x02, J9 Conn_01x02, Q3 BC547, Q4 IRLZ44N

Commit message: PCB v2.2
Other:
- board text added: "TU BRAKUJE REZYSTORA!!!!!!"
Changed lines of the file:
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@@
 			(drillshape 0)
 			(scaleselection 1)
-			(outputdirectory "gerber/")
+			(outputdirectory "C:/Users/Administrator/Desktop/Piezotester_PCB/")
 		)
 	)
@@
 		)
 		(property "Value" "R 1"
-			(at 0 1.82 90)
+			(at 0 -2.95 90)
 			(layer "F.Fab")
 			(effects
@@
 		(tags "capacitor")
 		(property "Reference" "C11"
-			(at 0 -1.85 0)
+			(at 0.06 2.08 0)
 			(layer "F.SilkS")
 			(effects
@@
 		(layer "Margin")
 	)
+	(gr_text "TU BRAKUJE REZYSTORA!!!!!!\n"
+		(at 23.34 85.97 0)
+		(layer "F.Cu")
+		(effects
+			(font
+				(size 1.5 1.5)
+				(thickness 0.3)
+				(bold yes)
+			)
+			(justify left bottom)
+		)
+	)
 	(gr_text "PIEZOTESTER V2.1\n"
 		(at 80 149 0)
@@
 	)
 	(segment
-		(start 93.26 80.84)
-		(end 93.26 85.14)
+		(start 82.02 88.185)
+		(end 82.02 86.98)
 		(width 1)
 		(layer "F.Cu")
@@
 	)
 	(segment
-		(start 96.12 79.53)
-		(end 94.57 79.53)
+		(start 83.865 88.185)
+		(end 82.02 88.185)
 		(width 1)
 		(layer "F.Cu")
@@
 	)
 	(segment
-		(start 83.865 88.185)
-		(end 82.02 88.185)
+		(start 85.72 96.42)
+		(end 85.76 96.38)
 		(width 1)
 		(layer "F.Cu")
@@
 	)
 	(segment
-		(start 85.72 96.42)
-		(end 85.76 96.38)
+		(start 94.7 86.58)
+		(end 94.7 87.88)
 		(width 1)
 		(layer "F.Cu")
@@
 	)
 	(segment
-		(start 82.02 88.185)
-		(end 79.515 88.185)
+		(start 84.05 84.95)
+		(end 86.58 84.95)
 		(width 1)
 		(layer "F.Cu")
@@
 	)
 	(segment
-		(start 93.26 85.14)
-		(end 94.7 86.58)
+		(start 93.26 80.84)
+		(end 93.26 85.14)
 		(width 1)
 		(layer "F.Cu")
@@
 	)
 	(segment
-		(start 85.76 92.24)
-		(end 85.77 92.23)
+		(start 94.57 79.53)
+		(end 93.26 80.84)
 		(width 1)
 		(layer "F.Cu")
@@
 	)
 	(segment
-		(start 94.7 86.58)
-		(end 94.7 87.88)
+		(start 82.02 88.185)
+		(end 79.515 88.185)
 		(width 1)
 		(layer "F.Cu")
@@
 	)
 	(segment
-		(start 85.76 96.38)
-		(end 85.76 92.24)
+		(start 85.76 92.24)
+		(end 85.77 92.23)
 		(width 1)
 		(layer "F.Cu")
@@
 	)
 	(segment
-		(start 85.77 92.23)
-		(end 85.77 90.09)
+		(start 85.76 96.38)
+		(end 85.76 92.24)
 		(width 1)
 		(layer "F.Cu")
@@
 	)
 	(segment
-		(start 85.72 101.65)
-		(end 85.72 96.42)
+		(start 85.77 92.23)
+		(end 85.77 90.09)
 		(width 1)
 		(layer "F.Cu")
@@
 	)
 	(segment
-		(start 82.02 88.185)
-		(end 82.02 86.98)
+		(start 82.02 86.98)
+		(end 84.05 84.95)
 		(width 1)
 		(layer "F.Cu")
@@
 	)
 	(segment
-		(start 85.77 90.09)
-		(end 83.865 88.185)
+		(start 85.72 101.65)
+		(end 85.72 96.42)
 		(width 1)
 		(layer "F.Cu")
@@
 	)
 	(segment
-		(start 84.05 84.95)
-		(end 86.58 84.95)
+		(start 96.12 79.53)
+		(end 94.57 79.53)
 		(width 1)
 		(layer "F.Cu")
@@
 	)
 	(segment
-		(start 82.02 86.98)
-		(end 84.05 84.95)
+		(start 93.26 85.14)
+		(end 94.7 86.58)
 		(width 1)
 		(layer "F.Cu")
@@
 	)
 	(segment
-		(start 94.57 79.53)
-		(end 93.26 80.84)
+		(start 85.77 90.09)
+		(end 83.865 88.185)
 		(width 1)
 		(layer "F.Cu")
