File: hardware/PCB/PCB V2.1/piezotesterV2.1/piezotesterV2.1.kicad_sch (KiCad schematic)
At the start: 49 parts, among them IC1 MCP6002-I_P, IC2 LM358P, IC3 LM2596S-5.0_NOPB, IC4 LP2950-33LPRE3, J1 Conn_01x02, J2 Conn_01x04, J8 Conn_01x02, J9 Conn_01x02, Q3 BC547, Q4 IRLZ44N

Commit message: PCB v2.2
Parts:
- added J10: Conn_01x02, Connector_PinHeader_2.54mm:PinHeader_1x02_P2.54mm_Horizontal, symbol Connector_Generic:Conn_01x02
- added Q7: BC337, Package_TO_SOT_THT:TO-92_Inline, symbol Transistor_BJT:BC547
- added Q8: IRLZ44N, Package_TO_SOT_THT:TO-220-3_Vertical, symbol Transistor_FET:IRLZ44N
- added R13: R 68K, Resistor_SMD:R_1206_3216Metric, symbol 1323:R
- added R17: R 100, Resistor_SMD:R_1206_3216Metric, symbol 1323:R
Connections:
- net 12VDC+: now also J10.1 (Pin_1), R13.1
- net GND: now also Q7.3 (E), Q8.3 (S)
- net GPIO17: now also R17.1
- new net: J10.2 (Pin_2), Q8.2 (D)
- new net: Q7.1 (C), Q8.1 (G), R13.2
- new net: Q7.2 (B), R17.2

Commit message: chore: sync repository with current workspace layout
Other:
- note removed: "SENSOR SECTION"
Changed lines of the file:
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@@
-		)
-	)
-	(text "SENSOR SECTION"
-		(exclude_from_sim no)
-		(at 196.85 20.32 0)
-		(effects
-			(font
-				(size 5.08 5.08)
-			)
 		)
 	)
